Commit message: New changes

File: src/first_robot/xacro/first_robot/first_robot.xacro (robot description, xacro)
@@ -18,5 +18,5 @@
     <inertial>
         <mass value="3.0"/>
-        <inertia ixx="0.0225" ixy="0.0" ixz="0.0" iyy="0.005625" iyz="0.0" izz="0.028125"/>
+        <inertia ixx="0.01" ixy="0.0" ixz="0.0" iyy="0.0225" iyz="0.0" izz="0.0325"/>
     </inertial>
   </link>
